Commit message: adds panda mjcf, scene for mjx

File: assets/descriptions/panda/urdf/panda.urdf (robot description, URDF)
Before this commit: robot panda, 12 links, 11 joints
Links:
- added link panda_hand_tcp
- added link panda_leftfinger_pad
- added link panda_rightfinger_pad
- link panda_hand: mass None -> 0.73; geometry collision mesh filename=franka_description/meshes/collision/hand.stl; visual mesh filename=franka_description/meshes/visual/hand.glb
- link panda_leftfinger: mass None -> 0.015; geometry collision box size=17.5e-3 15.2e-3 18.5e-3; collision box size=17.5e-3 7e-3 23.5e-3
- link panda_link0: mass None -> 0.629769; geometry collision mesh filename=franka_description/meshes/collision/link0.stl; visual mesh filename=franka_description/meshes/visual/link0.glb
- link panda_link1: mass None -> 4.970684; geometry collision mesh filename=franka_description/meshes/collision/link1.stl; visual mesh filename=franka_description/meshes/visual/link1.glb
- link panda_link2: mass None -> 0.646926; geometry collision mesh filename=franka_description/meshes/collision/link2.stl; visual mesh filename=franka_description/meshes/visual/link2.glb
- link panda_link3: mass None -> 3.228604; geometry collision mesh filename=franka_description/meshes/collision/link3.stl; visual mesh filename=franka_description/meshes/visual/link3.glb
- link panda_link4: mass None -> 3.587895; geometry collision mesh filename=franka_description/meshes/collision/link4.stl; visual mesh filename=franka_description/meshes/visual/link4.glb
- link panda_link5: mass None -> 1.225946; geometry collision mesh filename=franka_description/meshes/collision/link5.stl; visual mesh filename=franka_description/meshes/visual/link5.glb
- link panda_link6: mass None -> 1.666555; geometry collision mesh filename=franka_description/meshes/collision/link6.stl; visual mesh filename=franka_description/meshes/visual/link6.glb
- link panda_link7: mass None -> 0.735522; geometry collision mesh filename=franka_description/meshes/collision/link7.stl; visual mesh filename=franka_description/meshes/visual/link7.glb
- link panda_rightfinger: mass None -> 0.015; geometry collision box size=17.5e-3 15.2e-3 18.5e-3; collision box size=17.5e-3 7e-3 23.5e-3
Joints:
- added joint panda_hand_tcp_joint: type fixed, parent panda_hand, child panda_hand_tcp, origin xyz=0 0 0.1034 rpy=0 0 0
- added joint panda_leftfinger_pad_joint: type fixed, parent panda_leftfinger, child panda_leftfinger_pad, origin xyz=0 0 0.0455 rpy=0 0 0
- added joint panda_rightfinger_pad_joint: type fixed, parent panda_rightfinger, child panda_rightfinger_pad, origin xyz=0 0 0.0455 rpy=0 0 0
- joint panda_finger_joint1: limit lower=0.0 upper=0.04 effort=20 velocity=0.2 -> lower=0.0 upper=0.04 effort=100 velocity=0.2
- joint panda_finger_joint2: limit lower=0.0 upper=0.04 effort=20 velocity=0.2 -> lower=0.0 upper=0.04 effort=100 velocity=0.2
- joint panda_hand_joint: origin xyz=0 0 0 rpy=0 0 -0.785398163397 -> xyz=0 0 0 rpy=0 0 -0.7853981633974483
- joint panda_joint2: origin xyz=0 0 0 rpy=-1.57079632679 0 0 -> xyz=0 0 0 rpy=-1.5707963267948966 0 0
- joint panda_joint3: origin xyz=0 -0.316 0 rpy=1.57079632679 0 0 -> xyz=0 -0.316 0 rpy=1.5707963267948966 0 0
- joint panda_joint4: origin xyz=0.0825 0 0 rpy=1.57079632679 0 0 -> xyz=0.0825 0 0 rpy=1.5707963267948966 0 0
- joint panda_joint5: origin xyz=-0.0825 0.384 0 rpy=-1.57079632679 0 0 -> xyz=-0.0825 0.384 0 rpy=-1.5707963267948966 0 0
- joint panda_joint6: origin xyz=0 0 0 rpy=1.57079632679 0 0 -> xyz=0 0 0 rpy=1.5707963267948966 0 0
- joint panda_joint7: origin xyz=0.088 0 0 rpy=1.57079632679 0 0 -> xyz=0.088 0 0 rpy=1.5707963267948966 0 0
- joint panda_joint8: axis 0 0 0 -> (none)
