Commit message: almost there

File: source/tritonhumanoid/tritonhumanoid/assets/human_offset.urdf (robot description, URDF)
Before this commit: robot ch_robot, 12 links, 11 joints
Joints:
- joint left_ankle_joint: limit lower=-1.57 upper=1.57 effort=100 velocity=5.0 -> lower=-0.6 upper=0.6 effort=100 velocity=5.0
- joint left_hip2_joint: limit lower=-1.57 upper=1.57 effort=100 velocity=5.0 -> lower=-1.57 upper=0.436332 effort=100 velocity=5.0
- joint left_knee_joint: limit lower=-1.57 upper=1.57 effort=100 velocity=5.0 -> lower=-2.0944 upper=0 effort=100 velocity=5.0
- joint left_thigh_joint: limit lower=-1.57 upper=1.57 effort=100 velocity=5.0 -> lower=-0.785398 upper=0.785398 effort=100 velocity=5.0
- joint right_ankle_joint: limit lower=-1.57 upper=1.57 effort=100 velocity=5.0 -> lower=-0.6 upper=0.6 effort=100 velocity=5.0
- joint right_hip2_joint: limit lower=-1.57 upper=1.57 effort=100 velocity=5.0 -> lower=-0.436332 upper=1.57 effort=100 velocity=5.0
- joint right_knee_joint: limit lower=-1.57 upper=1.57 effort=100 velocity=5.0 -> lower=-2.0944 upper=0 effort=100 velocity=5.0
- joint right_thigh_joint: limit lower=-1.57 upper=1.57 effort=100 velocity=5.0 -> lower=-0.785398 upper=0.785398 effort=100 velocity=5.0

Commit message: progress save

File: source/tritonhumanoid/tritonhumanoid/assets/human_offset.urdf (robot description, URDF)
Before this commit: robot ch_robot, 12 links, 11 joints
Links:
- added link torso, mass 10.0; collision box size=0.32 0.16 0.24; visual box size=0.32 0.16 0.24
- link hip: mass 0.1 -> 5.159055
- link left_foot: mass 0.1 -> 0.765723
- link left_leg1: mass 0.1 -> 2.189611
- link left_leg2: mass 0.1 -> 1.709674
- link left_leg3: mass 0.1 -> 3.156742
- link left_leg4: mass 0.1 -> 1.980828
- link right_foot: mass 0.1 -> 0.765723
- link right_leg1: mass 0.1 -> 2.189548
- link right_leg2: mass 0.1 -> 1.72284
- link right_leg3: mass 0.1 -> 3.074969
- link right_leg4: mass 0.1 -> 1.980828
Joints:
- added joint hip_to_torso: type fixed, parent hip, child torso, origin xyz=-0.155 -0.03 0.765 rpy=0 0 0
- joint base_to_hip: origin xyz=0.157 0.03 -0.6 rpy=0 0 0 -> xyz=0 0 0 rpy=0 0 0

Commit message: updated humanoid model

File: source/tritonhumanoid/tritonhumanoid/assets/human_offset.urdf (robot description, URDF)
Before this commit: robot ch_robot, 13 links, 12 joints
Links:
- added link world
- link left_foot: geometry collision box size=0.08 0.21 0.01526; visual mesh filename=robot_meshes/visual/left_foot.stl scale=0.001 0.001 0.001
- link right_foot: geometry collision box size=0.08 0.21 0.01526; visual mesh filename=robot_meshes/visual/right_foot.stl scale=0.001 0.001 0.001
- link torso: mass 10.0 -> 3.175; geometry collision box size=0.28 0.12 0.096; visual mesh filename=robot_meshes/visual/battery_box.stl scale=0.001 0.001 0.001
Joints:
- added joint world_to_base: type fixed, parent world, child base_link, origin xyz=0.155 0.03 -0.765 rpy=0 0 0
- joint hip_to_torso: origin xyz=-0.155 -0.03 0.765 rpy=0 0 0 -> xyz=0 0 0 rpy=0 0 0

Commit message: updated thigh joint to be inverted

File: source/tritonhumanoid/tritonhumanoid/assets/human_offset.urdf (robot description, URDF)
Before this commit: robot ch_robot, 14 links, 13 joints
Joints:
- joint left_thigh_joint: axis 0.0 0.0 1.0 -> 0.0 0.0 -1.0
