Commit message: updated urdf

File: source/tritonhumanoid/tritonhumanoid/assets/human_offset_nf.urdf (robot description, URDF)
Before this commit: robot ch_robot, 14 links, 13 joints
Links:
- removed link base_link
Joints:
- removed joint base_to_hip
- removed joint hip_to_torso
- added joint torso_to_hip: type fixed, parent torso, child hip, origin xyz=0 0 0 rpy=0 0 0
- joint world_to_base: child base_link -> torso
