Commit message: yuh

File: source/tritonhumanoid/tritonhumanoid/assets/human_offset_corrected.urdf (robot description, URDF)
Before this commit: robot ch_robot, 13 links, 12 joints
Joints:
- joint world_to_base: origin xyz=0.155 0.03 -0.765 rpy=0 0 0 -> xyz=0.155 0.016 -0.63 rpy=0 0 0

Commit message: updated imu and model

File: source/tritonhumanoid/tritonhumanoid/assets/human_offset_corrected.urdf (robot description, URDF)
Before this commit: robot ch_robot, 13 links, 12 joints
Links:
- link torso: mass 3.175 -> 4.646; geometry collision cylinder length=0.02279 radius=0.105; visual mesh filename=robot_meshes/visual/imu_mount.stl scale=0.001 0.001 0.001
Joints:
- joint world_to_base: origin xyz=0.155 0.016 -0.63 rpy=0 0 0 -> xyz=0.1505 0.008 -0.6996 rpy=0 0 0

File: source/tritonhumanoid/tritonhumanoid/assets/human_offset_nf.urdf (robot description, URDF)
Before this commit: robot ch_robot, 13 links, 12 joints
Links:
- link torso: mass 3.175 -> 4.646; geometry collision cylinder length=0.011395 radius=0.105; visual mesh filename=robot_meshes/visual/imu_mount.stl scale=0.001 0.001 0.001

Commit message: update for motion tracking training

File: source/tritonhumanoid/tritonhumanoid/assets/human_offset_corrected.urdf (robot description, URDF)
Before this commit: robot ch_robot, 13 links, 12 joints
Links:
- link hip: geometry visual mesh filename=robot_meshes/visual/hip_dumb2.stl scale=0.001 0.001 0.001
- link left_leg1: geometry visual mesh filename=robot_meshes/visual/left_leg1_dumb.stl scale=0.001 0.001 0.001
- link left_leg2: geometry visual mesh filename=robot_meshes/visual/left_leg2_dumb.stl scale=0.001 0.001 0.001
- link left_leg3: geometry visual mesh filename=robot_meshes/visual/left_leg3_dumb.stl scale=0.001 0.001 0.001
- link left_leg4: geometry visual mesh filename=robot_meshes/visual/left_leg4_dumb.stl scale=0.001 0.001 0.001
- link right_leg1: geometry visual mesh filename=robot_meshes/visual/right_leg1_dumb.stl scale=0.001 0.001 0.001
- link right_leg2: geometry visual mesh filename=robot_meshes/visual/right_leg2_dumb.stl scale=0.001 0.001 0.001
- link right_leg3: geometry visual mesh filename=robot_meshes/visual/right_leg3_dumb.stl scale=0.001 0.001 0.001
- link right_leg4: geometry visual mesh filename=robot_meshes/visual/right_leg4_dumb.stl scale=0.001 0.001 0.001
- link torso: geometry visual mesh filename=robot_meshes/visual/imu_mount.stl scale=0.001 0.001 0.001; visual mesh filename=robot_meshes/visual/torso_weight.stl scale=0.001 0.001 0.001
